File: ECAD/i2c-master/i2c-master.kicad_pcb (KiCad board)
At the start: 2 copper layers, 40 x 36.8 mm, 18 parts, among them J1 Conn_01x12_Female, J10 Conn_01x04, J11 Barrel_Jack, J12 Conn_02x10_Odd_Even, J2 Conn_01x04, J3 Conn_01x04, J4 Conn_01x04, J5 Conn_01x04, J6 Conn_01x12_Female, J7 Conn_01x04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

Commit message: Change from 1x04 2.54mm headers to 1x05 micro JST
Parts:
- J10, J2, J3, J4, J5, J7, J8, J9: value Conn_01x04 -> Conn_01x05; footprint Connector_PinHeader_2.54mm:PinHeader_1x04_P2.54mm_Vertical -> Connector_JST:JST_GH_BM05B-GHS-TBT_1x05-1MP_P1.25mm_Vertical
- moved J8 11.4 mm to (35.1, 49.8)
- moved J10 10.6 mm to (35.1, 64.0)
- moved J3 10.2 mm to (46.2, 49.8)
- moved H1 9.65 mm to (33.5, 35.6)
- moved J7 9.62 mm to (35.1, 42.7)
- moved J9 9.45 mm to (35.1, 56.9)
- moved J5 9.33 mm to (46.2, 64.0)
- moved J2 2.87 mm to (46.2, 42.7)
- moved J4 2.27 mm to (46.2, 56.9)
- renumbered JP1 to 5V
Connections:
- J10 pad 4: GND -> IO4-A6
- J2 pad 4: GND -> IO4-A6
- J3 pad 4: GND -> IO4-A6
- J4 pad 4: GND -> IO4-A6
- J5 pad 4: GND -> IO4-A6
- J7 pad 4: GND -> IO4-A6
- J8 pad 4: GND -> IO4-A6
- J9 pad 4: GND -> IO4-A6
Routing:
- net IO4-A6: track 21.7 -> 92.0 mm, vias 1 -> 3
- net !IO3-SCL: track 67.6 -> 103.2 mm, vias 0 -> 2
- net +5V: track 48.8 -> 76.4 mm, vias 1 -> 3
- net IO2-SDA: track 62.5 -> 88.9 mm, vias 0 -> 2
- net GND: track 17.8 -> 42.7 mm, vias 13 -> 10
Other:
- board size 40 x 36.8 mm -> 49.9 x 36.8 mm
- board text removed: "5V"
- board text removed: "GND 5V"

Commit message: Whoops, forgot the master board
Parts:
- J10, J2, J3, J4, J5, J7, J8, J9: value Conn_01x05 -> Conn_01x04; footprint Connector_JST:JST_GH_BM05B-GHS-TBT_1x05-1MP_P1.25mm_Vertical -> Connector_JST:JST_GH_BM04B-GHS-TBT_1x04-1MP_P1.25mm_Vertical
- moved J2 11.8 mm to (34.4, 42.7)
- moved J3 11.8 mm to (34.4, 49.8)
- moved J4 11.8 mm to (34.4, 56.9)
- moved J5 11.8 mm to (34.4, 64.0)
- moved J10 10.5 mm to (45.6, 64.0)
- moved J7 10.5 mm to (45.6, 42.7)
- moved J8 10.5 mm to (45.6, 49.8)
- moved J9 10.5 mm to (45.6, 56.9)
- renumbered 5V to JP1
Connections:
- J10 pad 4: IO4-A6 -> GND
- J2 pad 4: IO4-A6 -> GND
- J3 pad 4: IO4-A6 -> GND
- J4 pad 4: IO4-A6 -> GND
- J5 pad 4: IO4-A6 -> GND
- J7 pad 4: IO4-A6 -> GND
- J8 pad 4: IO4-A6 -> GND
- J9 pad 4: IO4-A6 -> GND
Routing:
- net IO4-A6: track 92.0 -> 21.7 mm, vias 3 -> 1
- net GND: track 42.7 -> 0.00 mm
- net IO2-SDA: track 88.9 -> 88.1 mm

Commit message: 5-pin -> 4-pin JST
Parts:
- renumbered JP1 to 5V
